File: Debug_BreakBoard.kicad_pcb (KiCad board)
At the start: 2 copper layers, 97 x 26 mm, 69 parts, among them J1 FFC2A32-12-T, J10 Conn_01x03_Pin, J11 Conn_01x03_Pin, J12 Conn_01x03_Pin, J13 Conn_01x03_Pin, J14 Conn_01x03_Pin, J15 Conn_01x03_Pin, J16 Conn_01x03_Pin, J2 Conn_02x12_Counter_Clockwise, J3 Conn_01x03_Pin, J4 Conn_02x12_Counter_Clockwise, J5 Conn_01x03_Pin, J6 Conn_01x03_Pin, J7 Conn_01x03_Pin, J8 Conn_02x12_Counter_Clockwise, J9 Conn_01x03_Pin, P1 USB4125-GF-A-0190, SW1 SW_Push, SW10 SW_Push, SW11 SW_Push, SW12 SW_Push, SW2 SW_Push, SW3 SW_Push, SW4 SW_Push, SW5 SW_Push, SW6 SW_Push, SW7 SW_Push, SW8 SW_Push, SW9 SW_Push, U1 TLV6001UIDBVR, U10 TLV6001UIDBVR, U11 TLV6001UIDBVR, U12 TLV6001UIDBVR, U2 TLV6001UIDBVR, U3 TLV6001UIDBVR, U4 TLV6001UIDBVR, U5 TLV6001UIDBVR, U6 TLV6001UIDBVR, U7 TLV6001UIDBVR, U8 TLV6001UIDBVR, U9 TLV6001UIDBVR

Commit message: done
Parts:
- moved D1 56.8 mm to (124.2, 49.0)
- moved D10 56.8 mm to (124.2, 67.0)
- moved D11 56.8 mm to (124.2, 69.0)
- moved D12 56.8 mm to (124.2, 71.0)
- moved D2 56.8 mm to (124.2, 51.0)
- moved D3 56.8 mm to (124.2, 53.0)
- moved D4 56.8 mm to (124.2, 55.0)
- moved D5 56.8 mm to (124.2, 57.0)
- moved D6 56.8 mm to (124.2, 59.0)
- moved D7 56.8 mm to (124.2, 61.0)
- moved D8 56.8 mm to (124.2, 63.0)
- moved D9 56.8 mm to (124.2, 65.0)
- moved R1 56.8 mm to (120.2, 49.0)
- moved R10 56.8 mm to (120.2, 67.0)
- moved R11 56.8 mm to (120.2, 69.0)
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Connections:
- H1 pad 1: GND -> unconnected-(H1-Pad1)
- H2 pad 1: GND -> unconnected-(H2-Pad1)
- H3 pad 1: GND -> unconnected-(H3-Pad1)
- H4 pad 1: GND -> unconnected-(H4-Pad1)
- J1 pad S1: GND -> unconnected-(J1-SHIELD-PadS1)
- J1 pad S2: GND -> unconnected-(J1-SHIELD-PadS1)
- J1 pad S3: GND -> unconnected-(J1-SHIELD-PadS1)
- J1 pad S4: GND -> unconnected-(J1-SHIELD-PadS1)
- R10 pad 1: Net-(U10--) -> Net-(U11--)
- R11 pad 1: Net-(U11--) -> Net-(U6--)
- R2 pad 1: Net-(U2--) -> Net-(U7--)
- R3 pad 1: Net-(U3--) -> Net-(U2--)
- R4 pad 1: Net-(U4--) -> Net-(U8--)
- R5 pad 1: Net-(U5--) -> Net-(U3--)
- R6 pad 1: Net-(U6--) -> Net-(U9--)
- R7 pad 1: Net-(U7--) -> Net-(U4--)
- R8 pad 1: Net-(U8--) -> Net-(U10--)
- R9 pad 1: Net-(U9--) -> Net-(U5--)
- SW1 pad 2: /1 -> /7
- SW10 pad 2: /10 -> /4
- SW11 pad 2: /11 -> /5
- SW12 pad 2: /12 -> /6
- SW2 pad 2: /2 -> /8
- SW3 pad 2: /3 -> /9
- SW4 pad 2: /4 -> /10
- SW5 pad 2: /5 -> /11
- SW6 pad 2: /6 -> /12
- SW7 pad 2: /7 -> /1
- SW8 pad 2: /8 -> /2
- SW9 pad 2: /9 -> /3
- U10 pad 3: /10 -> /8
- U11 pad 3: /11 -> /10
- U2 pad 3: /2 -> /3
- U3 pad 3: /3 -> /5
- U4 pad 3: /4 -> /7
- U5 pad 3: /5 -> /9
- U6 pad 3: /6 -> /11
- U7 pad 3: /7 -> /2
- U8 pad 3: /8 -> /4
- U9 pad 3: /9 -> /6
Routing:
- net VDD: track 0.00 -> 151.3 mm
- net /12: track 0.00 -> 112.8 mm, vias 0 -> 3
- net /10: track 0.00 -> 101.9 mm, vias 0 -> 1
- net /2: track 0.00 -> 101.4 mm, vias 0 -> 1
- net /4: track 0.00 -> 100.0 mm, vias 0 -> 1
- net /8: track 0.00 -> 97.5 mm, vias 0 -> 1
- net /1: track 0.00 -> 97.4 mm
- net /6: track 0.00 -> 97.0 mm, vias 0 -> 2
- net /11: track 0.00 -> 95.7 mm
- net /3: track 0.00 -> 94.3 mm
- net /9: track 0.00 -> 92.8 mm
- net /5: track 0.00 -> 90.7 mm
- net /7: track 0.00 -> 89.4 mm
- net P5V0: track 0.00 -> 18.3 mm, vias 0 -> 16
- net GND: track 0.00 -> 14.0 mm, vias 0 -> 12
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- added copper zone on B.Cu, net GND
- added copper zone on F.Cu, net GND
- added copper zone on B.Cu, net P5V0
Other:
- outline, holes or cut-outs redrawn
- board text added: "BTN"
- board text added: "CHOOSE GND PIN HERE"
- board text added: "CHOOSE VCC PIN HERE"
- board text added: "DEBUG BREAKBOARD rev 1.0"
- board text added: "GND"
- board text added: "VDD"
- board text added: "You must choose GND, but not VDD. You can use VDD to connect to another pin and it will become common for all buttons."

Commit message: update
Parts:
- added J17: Conn_01x02_Pin, Connector_PinHeader_2.54mm:PinHeader_1x02_P2.54mm_Vertical, F.Cu at (105.9, 58.5)
- moved J10 9.50 mm to (177.7, 61.5)
- moved J11 9.50 mm to (140.7, 58.5)
- moved J12 9.50 mm to (147.7, 58.5)
- moved J13 9.50 mm to (155.7, 58.5)
- moved J14 9.50 mm to (162.7, 58.5)
- moved J15 9.50 mm to (170.7, 58.5)
- moved J16 9.50 mm to (177.7, 58.5)
- moved J3 9.50 mm to (140.7, 61.5)
- moved J5 9.50 mm to (147.7, 61.5)
- moved J6 9.50 mm to (155.7, 61.5)
- moved J7 9.50 mm to (162.7, 61.5)
- moved J9 9.50 mm to (170.7, 61.5)
- moved P1 3.50 mm to (99.0, 60.0)
- moved H1 3.00 mm to (100.0, 50.0)
- moved H2 3.00 mm to (100.0, 70.0)
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Routing:
- net VDD: track 151.3 -> 101.8 mm
- net /12: track 112.8 -> 101.4 mm, vias 3 -> 1
- net /7: track 89.4 -> 94.4 mm
- net /8: track 97.5 -> 101.1 mm
- net /9: track 92.8 -> 94.2 mm
- net /6: track 97.0 -> 98.2 mm, vias 2 -> 1
- net /11: track 95.7 -> 94.6 mm
- net /2: track 101.4 -> 102.0 mm
- net Net-(U2--): track 7.37 -> 6.84 mm
- net Net-(U9--): track 12.4 -> 11.9 mm
- net Net-(U8--): track 12.3 -> 11.8 mm
- net Net-(U12--): track 12.3 -> 11.8 mm
- net Net-(U11--): track 12.4 -> 11.9 mm
- net Net-(U10--): track 12.4 -> 11.9 mm
Other:
- board size 97 x 26 mm -> 100 x 26 mm
- board text added: "5V"

Commit message: bom
Parts:
- J10, J11, J12, J13, J14, J15, J16, J3, J5, J6, J7, J9: footprint Connector_PinHeader_2.00mm:PinHeader_1x03_P2.00mm_Vertical -> Connector_PinHeader_2.54mm:PinHeader_1x03_P2.54mm_Vertical
- J2, J4, J8: footprint Connector_PinHeader_2.00mm:PinHeader_2x12_P2.00mm_Vertical -> Connector_PinHeader_2.54mm:PinHeader_2x12_P2.54mm_Vertical
- moved J3 6.12 mm to (139.5, 67.5)
- moved J6 6.06 mm to (154.9, 67.5)
- moved R12 6.03 mm to (119.2, 76.9)
- moved J5 6.02 mm to (147.2, 67.5)
- moved J9 6.02 mm to (170.3, 67.5)
- moved J10 6.01 mm to (178.0, 67.5)
- moved J7 6.00 mm to (162.6, 67.5)
- moved H2 6.00 mm to (100.0, 76.0)
- moved H4 6.00 mm to (194.0, 76.0)
- moved SW1 6.00 mm to (140.2, 77.0)
- moved SW2 6.00 mm to (147.7, 77.0)
- moved SW3 6.00 mm to (155.2, 77.0)
- moved SW4 6.00 mm to (162.7, 77.0)
- moved SW5 6.00 mm to (170.2, 77.0)
- moved SW6 6.00 mm to (177.8, 77.0)
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Routing:
- net VDD: track 101.8 -> 0.00 mm
- net GND: track 14.0 -> 32.7 mm, vias 12 -> 30
- net P5V0: track 18.3 -> 4.69 mm
- net /5: track 90.7 -> 102.7 mm
- net /6: track 98.2 -> 105.5 mm
- net /11: track 94.6 -> 99.8 mm
- net /9: track 94.2 -> 98.8 mm
- net /8: track 101.1 -> 105.5 mm
- net /7: track 94.4 -> 98.4 mm
- net /12: track 101.4 -> 104.5 mm
- net /1: track 97.3 -> 100.3 mm
- net /2: track 102.0 -> 104.9 mm
- net /4: track 100.5 -> 103.4 mm
- net /3: track 94.5 -> 97.2 mm
- net /10: track 101.5 -> 103.7 mm
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- added copper zone on In1.Cu, net GND
- added copper zone on In2.Cu, net VDD
- removed copper zone on B.Cu, net GND
- removed copper zone on F.Cu, net GND
Other:
- board size 100 x 26 mm -> 100 x 32 mm
- copper layers 2 -> 4
