File: Debug_BreakBoard.kicad_sch (KiCad schematic)
At the start: 69 parts, among them J1 FFC2A32-12-T, J10 Conn_01x03_Pin, J11 Conn_01x03_Pin, J12 Conn_01x03_Pin, J13 Conn_01x03_Pin, J14 Conn_01x03_Pin, J15 Conn_01x03_Pin, J16 Conn_01x03_Pin, J2 Conn_02x12_Counter_Clockwise, J3 Conn_01x03_Pin, J4 Conn_02x12_Counter_Clockwise, J5 Conn_01x03_Pin, J6 Conn_01x03_Pin, J7 Conn_01x03_Pin, J8 Conn_02x12_Counter_Clockwise, J9 Conn_01x03_Pin, P1 USB4125-GF-A-0190, SW1 SW_Push, SW10 SW_Push, SW11 SW_Push, SW12 SW_Push, SW2 SW_Push, SW3 SW_Push, SW4 SW_Push, SW5 SW_Push, SW6 SW_Push, SW7 SW_Push, SW8 SW_Push, SW9 SW_Push, U1 TLV6001UIDBVR, U10 TLV6001UIDBVR, U11 TLV6001UIDBVR, U12 TLV6001UIDBVR, U2 TLV6001UIDBVR, U3 TLV6001UIDBVR, U4 TLV6001UIDBVR, U5 TLV6001UIDBVR, U6 TLV6001UIDBVR, U7 TLV6001UIDBVR, U8 TLV6001UIDBVR, U9 TLV6001UIDBVR

Commit message: done
Connections:
- net 1: now also SW7.2; no longer SW1.2
- net 10: now also SW4.2, U11.3 (+); no longer SW10.2, U10.3 (+)
- net 11: now also SW5.2, U6.3 (+); no longer SW11.2, U11.3 (+)
- net 12: now also SW6.2; no longer SW12.2
- net 2: now also SW8.2, U7.3 (+); no longer SW2.2, U2.3 (+)
- net 3: now also SW9.2, U2.3 (+); no longer SW3.2, U3.3 (+)
- net 4: now also SW10.2, U8.3 (+); no longer SW4.2, U4.3 (+)
- net 5: now also SW11.2, U3.3 (+); no longer SW5.2, U5.3 (+)
- net 6: now also SW12.2, U9.3 (+); no longer SW6.2, U6.3 (+)
- net 7: now also SW1.2, U4.3 (+); no longer SW7.2, U7.3 (+)
- net 8: now also SW2.2, U10.3 (+); no longer SW8.2, U8.3 (+)
- net 9: now also SW3.2, U5.3 (+); no longer SW9.2, U9.3 (+)
- net GND: no longer H1.1, H2.1, H3.1, H4.1, J1.S1 (SHIELD), J1.S2 (SHIELD), J1.S3 (SHIELD), J1.S4 (SHIELD)
- net at U11.1, U11.4 (-): now also R10.1; no longer R11.1
- net at U2.1, U2.4 (-): now also R3.1; no longer R2.1
- net at U8.1, U8.4 (-): now also R4.1; no longer R8.1
- net at U9.1, U9.4 (-): now also R6.1; no longer R9.1
- net at U4.1, U4.4 (-): now also R7.1; no longer R4.1
- net at U3.1, U3.4 (-): now also R5.1; no longer R3.1
- net at U10.1, U10.4 (-): now also R8.1; no longer R10.1
- net at U6.1, U6.4 (-): now also R11.1; no longer R6.1
- net at U7.1, U7.4 (-): now also R2.1; no longer R7.1
- net at U5.1, U5.4 (-): now also R9.1; no longer R5.1
- new net: J1.S1 (SHIELD), J1.S2 (SHIELD), J1.S3 (SHIELD), J1.S4 (SHIELD)
- no-connect marks 2 -> 7
Other:
- moved on the sheet: U10, U11, U2, U3, U4, U5, U6, U7, U8, U9

Commit message: update
Parts:
- added J17: Conn_01x02_Pin, Connector_PinHeader_2.54mm:PinHeader_1x02_P2.54mm_Vertical, symbol Connector:Conn_01x02_Pin
Connections:
- net GND: now also J17.2 (Pin_2)
- net P5V0: now also J17.1 (Pin_1)
Changed lines of the file:
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@@
     (stroke (width 0) (type default))
   )
+  (wire (pts (xy 217.17 255.27) (xy 219.71 255.27))
+    (stroke (width 0) (type default))
+  )
   (wire (pts (xy 43.18 44.45) (xy 45.72 44.45))
     (stroke (width 0) (type default))
@@
     (stroke (width 0) (type default))
   )
+  (wire (pts (xy 219.71 257.81) (xy 219.71 260.35))
+    (stroke (width 0) (type default))
+  )
   (wire (pts (xy 43.18 26.67) (xy 45.72 26.67))
     (stroke (width 0) (type default))
@@
     (stroke (width 0) (type default))
   )
+  (wire (pts (xy 217.17 257.81) (xy 219.71 257.81))
+    (stroke (width 0) (type default))
+  )
   (wire (pts (xy 393.7 58.42) (xy 396.24 58.42))
     (stroke (width 0) (type default))
@@
     (stroke (width 0) (type default))
   )
+  (wire (pts (xy 219.71 255.27) (xy 219.71 252.73))
+    (stroke (width 0) (type default))
+  )
   (wire (pts (xy 393.7 27.94) (xy 396.24 27.94))
     (stroke (width 0) (type default))
@@
     )
   )
+  (symbol (lib_id "Connector:Conn_01x02_Pin") (at 212.09 255.27 0) (unit 1)
+    (in_bom yes) (on_board yes) (dnp no) (fields_autoplaced)
+    (property "Reference" "J17" (at 212.725 252.73 0)
+      (effects (font (size 1.27 1.27)))
+    )
+    (property "Value" "Conn_01x02_Pin" (at 212.725 252.73 0)
+      (effects (font (size 1.27 1.27)) hide)
+    )
+    (property "Footprint" "Connector_PinHeader_2.54mm:PinHeader_1x02_P2.54mm_Vertical" (at 212.09 255.27 0)
+      (effects (font (size 1.27 1.27)) hide)
+    )
+    (property "Datasheet" "~" (at 212.09 255.27 0)
+      (effects (font (size 1.27 1.27)) hide)
+    )
+    (pin "1")
+    (pin "2")
+    (instances
+      (project "Debug_BreakBoard"
+        (path "/2138d703-2e6f-4ba3-855d-1f96478cf691"
+          (reference "J17") (unit 1)
+        )
+      )
+    )
+  )
   (symbol (lib_id "Switch:SW_Push") (at 120.65 185.42 0) (unit 1)
     (in_bom yes) (on_board yes) (dnp no) (fields_autoplaced)
@@
     )
   )
+  (symbol (lib_id "power:GND") (at 219.71 260.35 0) (unit 1)
+    (in_bom yes) (on_board yes) (dnp no) (fields_autoplaced)
+    (property "Reference" "#PWR01" (at 219.71 266.7 0)
+      (effects (font (size 1.27 1.27)) hide)
+    )
+    (property "Value" "GND" (at 219.71 265.43 0)
+      (effects (font (size 1.27 1.27)))
+    )
+    (property "Footprint" "" (at 219.71 260.35 0)
+      (effects (font (size 1.27 1.27)) hide)
+    )
+    (property "Datasheet" "" (at 219.71 260.35 0)
+      (effects (font (size 1.27 1.27)) hide)
+    )
+    (pin "1")
+    (instances
+      (project "Debug_BreakBoard"
+        (path "/2138d703-2e6f-4ba3-855d-1f96478cf691"
+          (reference "#PWR01") (unit 1)
+        )
+      )
+    )
+  )
   (symbol (lib_id "Connector:Conn_01x03_Pin") (at 57.15 116.84 0) (unit 1)
     (in_bom yes) (on_board yes) (dnp no) (fields_autoplaced)
@@
         )
       )
+    )
+  )
+  (symbol (lib_id "RackLab_PowerSymbols:P5V0") (at 219.71 252.73 0) (unit 1)
+    (in_bom yes) (on_board yes) (dnp no) (fields_autoplaced)
+    (property "Reference" "#PWR032" (at 219.71 256.54 0)
+      (effects (font (size 1.27 1.27)) hide)
+    )
+    (property "Value" "P5V0" (at 219.71 247.65 0)
+      (effects (font (size 1.27 1.27)))
+    )
+    (property "Footprint" "" (at 219.71 252.73 0)
+      (effects (font (size 1.27 1.27)) hide)
+    )
+    (property "Datasheet" "" (at 219.71 252.73 0)
+      (effects (font (size 1.27 1.27)) hide)
+    )
+    (pin "1")
+    (instances
+      (project "Debug_BreakBoard"
+        (path "/2138d703-2e6f-4ba3-855d-1f96478cf691"
+          (reference "#PWR032") (unit 1)
+        )
+      )

Commit message: bom
Parts:
- D1, D10, D11, D12, D2, D3, D4, D5, D6, D7, D8, D9: Manufacturer (none) -> Wurth Elektronik; Part Number (none) -> 150060BS75000
- H1, H2, H3, H4: now left out of the parts list
- J10, J11, J12, J13, J14, J15, J16, J3, J5, J6, J7, J9: footprint Connector_PinHeader_2.00mm:PinHeader_1x03_P2.00mm_Vertical -> Connector_PinHeader_2.54mm:PinHeader_1x03_P2.54mm_Vertical; Manufacturer (none) -> Amphenol FCI; Part Number (none) -> 68002-403HLF
- J2, J4, J8: footprint Connector_PinHeader_2.00mm:PinHeader_2x12_P2.00mm_Vertical -> Connector_PinHeader_2.54mm:PinHeader_2x12_P2.54mm_Vertical; Manufacturer (none) -> Amphenol FCI; Part Number (none) -> 10129381-924001BLF
- R1, R10, R11, R12, R2, R3, R4, R5, R6, R7, R8, R9: Manufacturer (none) -> Kamaya; Part Number (none) -> RMC1/16-511JTP
- SW1, SW10, SW11, SW12, SW2, SW3, SW4, SW5, SW6, SW7, SW8, SW9: Manufacturer (none) -> CUI Devices; Part Number (none) -> TS02-66-70-BK-100-SCR-D
